File: senior_design_pcb/senior_design_pcb.kicad_sch (KiCad schematic)
At the start: 0 parts

Commit message: updated chart
Other:
- note added: "(plus charge protection circuit)"
- note added: "Barrel Jack to PCB"
- note added: "LED on the comms for funny flashing light when programming?"
- note added: "Motors only signals go via pcb motor power cabled"
- note added: "Pi/Laptop/Jetson"
- note added: "battery pack"
- note added: "decoupling caps"
- note added: "motors"
- note added: "power"
- note added: "signals"
- note added: "these will all be 0805's"
- note removed: "Motor controls only signals go via pcb motor power cabled"
- note removed: "battery"
