File: hardware/senior_design_pcb/senior_design_pcb.kicad_sch (KiCad schematic)
At the start: 84 parts, among them J1 SBH11-PBPC-D05-ST-BK, J10 Screw_Terminal_01x05, J11 2x08Rectangle-LED Matrix Conn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, J12 1x05JST - Joystick2 connector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, J13 UJ20-C-H-C-4-SMT-TR, J2 Conn_01x08_Pin, J3 1x02JST-IR Transmitter1, J4 1x03JST- IR Receiver1, J5 1x05JST-Admin LCD Console Con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, J6 1x05JST - Joystick1 connector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

Commit message: updated pcb
shrunk edge cuts
added footprints for pnp
added new symbol for pnp
reorganized stm pinout for easier routing
moved connectors
Parts:
- removed J4: 1x03JST- IR Receiver1, Connector_JST:JST_EH_S3B-EH_1x03_P2.50mm_Horizontal, symbol Connector:Conn_01x03_Socket
- removed J7: 1x02JST-IR Transmitter, Connector_JST:JST_EH_S2B-EH_1x02_P2.50mm_Horizontal, symbol Connector:Conn_01x02_Socket
- removed J8: 1x03JST-IR Receiver2, Connector_JST:JST_EH_S3B-EH_1x03_P2.50mm_Horizontal, symbol Connector:Conn_01x03_Socket
- removed Q1, Q2, Q3, Q4, Q5, Q6: Q_PMOS_DGS, symbol Transistor_FET:Q_PMOS_DGS
- removed R14, R16: 75, symbol Device:R_US
- removed SW2, SW4: SW_Push, symbol Switch:SW_Push
- removed TP2: TestPoint, TestPoint:TestPoint_THTPad_D1.5mm_Drill0.7mm, symbol testpoint:TestPoint
- removed TP3: NRST, TestPoint:TestPoint_THTPad_D1.5mm_Drill0.7mm, symbol testpoint:TestPoint
- removed TP4: IR-IN1, TestPoint:TestPoint_THTPad_D1.5mm_Drill0.7mm, symbol testpoint:TestPoint
- removed TP5: IR-IN2, TestPoint:TestPoint_THTPad_D1.5mm_Drill0.7mm, symbol testpoint:TestPoint
- removed TP6: VBUS, TestPoint:TestPoint_THTPad_D1.5mm_Drill0.7mm, symbol testpoint:TestPoint
- removed TP7: +5V, TestPoint:TestPoint_THTPad_D1.5mm_Drill0.7mm, symbol testpoint:TestPoint
- removed TP8: 3V3, TestPoint:TestPoint_THTPad_D1.5mm_Drill0.7mm, symbol testpoint:TestPoint
- removed TP9: GND, TestPoint:TestPoint_THTPad_D1.5mm_Drill0.7mm, symbol testpoint:TestPoint
- removed XTAL1: 32.768kHz(12.5pF), Sr_ Design:ECS - CRYSTAL 32.7680KHZ 6PF SMD, symbol ECS-CRYSTAL 8MHZ 8PF SMD:ECS-80-8-33Q-ADS
- added C26: .1uF, Capacitor_SMD:C_0805_2012Metric_Pad1.18x1.45mm_HandSolder, symbol Device:C
- added D3: BAT60JFILM, Diode_SMD:D_SOD-323_HandSoldering, symbol Diode:BAT60A
- added J4: Conn_01x02_Socket, Connector_JST:JST_EH_B2B-EH-A_1x02_P2.50mm_Vertical, symbol Connector:Conn_01x02_Socket
- added R17: 1M, Resistor_SMD:R_0805_2012Metric_Pad1.20x1.40mm_HandSolder, symbol Device:R_US
- added U1, U5: USBLC6-2SC6Y, kicad_library:TVS-DIODE-USBLC6-2SC6Y, symbol TVS-DIODE-USBLC6-2SC6Y:USBLC6-2SC6Y
- added U6, U7, U8: 2SA1873-GRTE85L_F, kicad_library:TRANS 2PNP-2SA1873, symbol TRANS 2PNP-2SA1873:2SA1873-GRTE85L_F
- added XTAL1: ECX-.327-CDX-1293, kicad_library:32KHZ-CLK-ECX1293, symbol 32KHZ-CLK-ECX1293:ECX-.327-CDX-1293
- J10, J9: value Screw_Terminal_01x05 -> Conn_01x04_Socket; footprint Connector_JST:JST_EH_S6B-EH_1x06_P2.50mm_Horizontal -> Connector_JST:JST_EH_B4B-EH-A_1x04_P2.50mm_Vertical; symbol Connector:Screw_Terminal_01x05 -> Connector:Conn_01x04_Socket
- J12, J5, J6: footprint Connector_JST:JST_EH_S5B-EH_1x05_P2.50mm_Horizontal -> Connector_JST:JST_EH_B5B-EH-A_1x05_P2.50mm_Vertical
- J3: value 1x02JST-IR Transmitter1 -> Conn_01x02_Socket; footprint Connector_JST:JST_EH_S2B-EH_1x02_P2.50mm_Horizontal -> Connector_JST:JST_EH_B2B-EH-A_1x02_P2.50mm_Vertical
- R12: value 75 -> 10K; footprint (none) -> Resistor_SMD:R_0805_2012Metric_Pad1.20x1.40mm_HandSolder
Connections:
- net +5V: now also D3.1 (K), U1.5 (VBUS); no longer C2.1, FB1.1, J3.1 (Pin_1), R12.1
- net ADMIN_JOYSTICK-X: now also U2.9 (PC1); no longer U2.8 (PC0)
- net ADMIN_JOYSTICK-Y: now also U2.8 (PC0); no longer U2.9 (PC1)
- net DIR+1: now also J9.2 (Pin_2), U8.4; no longer J9.3 (Pin_3)
- net DIR+2: now also J10.2 (Pin_2), U6.5; no longer J10.3 (Pin_3)
- net ENA+1: now also J9.3 (Pin_3), U7.5; no longer J9.4 (Pin_4)
- net ENA+2: now also J10.3 (Pin_3), U6.4; no longer J10.4 (Pin_4)
- net GND: now also J10.4 (Pin_4), J9.4 (Pin_4), R12.2, C26.2, J4.2 (Pin_2), R17.2, U1.2 (GND), U5.2 (GND); no longer J10.5 (Pin_5), J9.5 (Pin_5)
- net HS_CLK-IN: now also C20.1, XTAL2.1; no longer C5.1
- net HS_CLK-OUT: now also C21.1, XTAL2.3; no longer C6.1
- net IR_IN_1: now also U1.4 (I/O2)
- net IR_IN_2: now also U1.6 (I/O1)
- net LS_CLK-IN: now also C5.1, XTAL1.1; no longer C20.1, XTAL2.1
- net LS_CLK-OUT: now also C6.1, XTAL1.2; no longer C21.1, XTAL2.3
- net PA0: no longer J2.7 (Pin_7)
- net PA1: no longer J2.8 (Pin_8)
- net PA8: now also U8.3
- net PA9: now also U8.1
- net PB5: no longer J2.1 (Pin_1)
- net PB6: no longer J2.2 (Pin_2)
- net PB7: no longer J2.3 (Pin_3)
- net PB8: no longer J2.4 (Pin_4)
- net PB9: no longer J2.5 (Pin_5)
- net PC3: no longer J2.6 (Pin_6)
- net PC6: now also U6.3
- net PC7: now also U6.1
- net PC8: now also U7.3
- net PC9: now also U7.1
- net PUL+1: now also J9.1 (Pin_1), U8.5; no longer J9.2 (Pin_2)
- net PUL+2: now also J10.1 (Pin_1), U7.4; no longer J10.2 (Pin_2)
- net VBUS: now also C26.1, U5.5 (VBUS)
- net usbc-shield: now also R17.1
- net at R15.2: now also U7.2
- net at R11.2: now also U6.2
- net at R13.2: now also U8.2
- net at FT1.11 (CTS): now also R12.1
- net D+ renamed Din +
- net Din +: now also U5.3 (I/O2); no longer FT1.16 (USBD-)
- net D- renamed Din -
- net Din -: now also U5.1 (I/O1); no longer FT1.15 (USBD+)
- new net: C2.1, D3.2 (A), FB1.1
- new net Dout+: FT1.16 (USBD-), U5.4 (I/O2)
- new net Dout-: FT1.15 (USBD+), U5.6 (I/O1)
- new net IR_IN_1-dir: J3.1 (Pin_1), U1.3 (I/O2)
- new net IR_IN_2-dir: J4.1 (Pin_1), U1.1 (I/O1)
- no-connect marks 21 -> 16
Other:
- note removed: "I_d < 16mA"
- note removed: "ill make this look prettier later"
- note removed: "in lab were using the pmos in the closet - will check the name tomorrow in lab"
- moved on the sheet: C10, C11, C12, C13, C14, C15, C16, C17, C18, C19, C20, C21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
