File: hardware/senior_design_pcb/senior_design_pcb.kicad_pcb (KiCad board)
At the start: 4 copper layers, 64.8 x 61.5 mm, 69 parts, among them J1 SBH11-PBPC-D05-ST-BK, J10 Conn_01x04_Socket, J11 2x08Rectangle-LED Matrix Conn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, J12 1x05JST - Joystick2 connector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, J13 UJ20-C-H-C-4-SMT-TR, J2 Conn_01x08_Pin, J3 Conn_01x02_Socket, J4 Conn_01x02_Socket, J5 1x05JST-Admin LCD Console Con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, J6 1x05JST - Joystick1 connector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

Commit message: routed more traces
just routed some more. oh and i also added an LED bc there was a pin i forgot we werent using anymore so like why not make it an on board led yk.
Parts:
- removed TP1: TestPoint_Small, TestPoint:TestPoint_Pad_D1.5mm
- added C27: .1uF, Capacitor_SMD:C_0805_2012Metric_Pad1.18x1.45mm_HandSolder, B.Cu at (82.5, 79.6)
- added C28: .1uF, Capacitor_SMD:C_0805_2012Metric_Pad1.18x1.45mm_HandSolder, B.Cu at (77.2, 79.6)
- added C29: .1uF, Capacitor_SMD:C_0805_2012Metric_Pad1.18x1.45mm_HandSolder, B.Cu at (87.5, 79.6)
- added H1: MountingHole, MountingHole:MountingHole_3.2mm_M3, F.Cu at (36.2, 48.2)
- added H2: MountingHole, MountingHole:MountingHole_3.2mm_M3, F.Cu at (36.2, 108.5)
- added H3: MountingHole, MountingHole:MountingHole_3.2mm_M3, F.Cu at (96.5, 48.2)
- added H4: MountingHole, MountingHole:MountingHole_3.2mm_M3, F.Cu at (96.5, 108.5)
- added LD3: LED_Red, LED_SMD:LED_0805_2012Metric, F.Cu at (44.3, 96.8)
- added LD4: LED_Red, LED_SMD:LED_0805_2012Metric, F.Cu at (67.8, 65.3)
- added LD5: LED_Yel, LED_SMD:LED_0805_2012Metric, F.Cu at (67.6, 58.9)
- added R11: 75, Resistor_SMD:R_0805_2012Metric_Pad1.20x1.40mm_HandSolder, B.Cu at (60.5, 60.0)
- added R13: 75, Resistor_SMD:R_0805_2012Metric_Pad1.20x1.40mm_HandSolder, B.Cu at (52.0, 60.0)
- added R14: 5k11, Resistor_SMD:R_0805_2012Metric_Pad1.20x1.40mm_HandSolder, F.Cu at (44.3, 94.0)
- added R15: 75, Resistor_SMD:R_0805_2012Metric_Pad1.20x1.40mm_HandSolder, B.Cu at (56.3, 60.0)
- added R16: 10K, Resistor_SMD:R_0805_2012Metric_Pad1.20x1.40mm_HandSolder, B.Cu at (82.5, 74.7)
- added R18: 10K, Resistor_SMD:R_0805_2012Metric_Pad1.20x1.40mm_HandSolder, B.Cu at (77.2, 74.7)
- added R19: 10K, Resistor_SMD:R_0805_2012Metric_Pad1.20x1.40mm_HandSolder, B.Cu at (87.5, 74.7)
- added R20: 68, Resistor_SMD:R_0805_2012Metric_Pad1.20x1.40mm_HandSolder, B.Cu at (67.8, 69.6)
- added R21: 68, Resistor_SMD:R_0805_2012Metric_Pad1.20x1.40mm_HandSolder, B.Cu at (67.4, 62.2)
- added U10: KMR241GLFS, General Library:KMR241G-RESET-BUTTON, F.Cu at (90.0, 77.1)
- added U9: KMR241GLFS, General Library:KMR241G-RESET-BUTTON, F.Cu at (79.8, 77.2)
- C14, C16: value 4.7uf -> 4.7uF; moved to B.Cu
- C22, C23, C25, R10, R3, R5, R6, R7, R9: moved to B.Cu
- U1: value USBLC6-2SC6Y -> KMR241GLFS; footprint kicad_library:TVS-DIODE-USBLC6-2SC6Y -> General Library:KMR241G-RESET-BUTTON
- moved C22 99.6 mm to (68.8, 98.5), turned to 0 degrees
- moved U4 92.4 mm to (67.0, 101.0), turned to 0 degrees
- moved R7 88.1 mm to (67.2, 88.7), turned to 90 degrees
- moved R6 86.6 mm to (64.8, 98.5), turned to 0 degrees
- moved LD2 53.3 mm to (46.5, 59.0), turned to 180 degrees
- moved LD1 50.3 mm to (46.5, 56.0), turned to 180 degrees
- moved R5 48.3 mm to (41.8, 59.0)
- moved U1 42.9 mm to (84.9, 77.1), turned to 90 degrees
- moved J3 37.5 mm to (79.0, 50.5), turned to 180 degrees
- moved J4 37.4 mm to (89.0, 50.5), turned to 180 degrees
- moved C26 19.4 mm to (44.2, 91.2)
- moved U7 13.3 mm to (57.4, 56.6)
- moved U8 13.3 mm to (53.0, 56.6)
- moved U6 13.3 mm to (61.4, 56.6)
- moved R9 9.54 mm to (94.0, 75.2)
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Connections:
- J10 pad 1: /PUL+2 -> GND
- J10 pad 2: /DIR+2 -> /ENA+2
- J10 pad 3: /ENA+2 -> /DIR+2
- J10 pad 4: GND -> /PUL+2
- J2 pad 1: unconnected-(J2-Pin_1-Pad1) -> +3V3
- J2 pad 2: unconnected-(J2-Pin_2-Pad2) -> /PB3
- J2 pad 3: unconnected-(J2-Pin_3-Pad3) -> /PB5
- J2 pad 4: unconnected-(J2-Pin_4-Pad4) -> /PB6
- J2 pad 5: unconnected-(J2-Pin_5-Pad5) -> /PB7
- J2 pad 6: unconnected-(J2-Pin_6-Pad6) -> /PB8
- J2 pad 7: unconnected-(J2-Pin_7-Pad7) -> /PB9
- J2 pad 8: unconnected-(J2-Pin_8-Pad8) -> GND
- J3 pad 1: /IR_IN_1-dir -> GND
- J3 pad 2: GND -> /IR_IN_1
- J4 pad 1: /IR_IN_2-dir -> GND
- J4 pad 2: GND -> /IR_IN_2
- J5 pad 1: +3V3 -> GND
- J5 pad 2: /CONSOLE_DISP-1 -> /CONSOLE_DISP-3
- J5 pad 4: /CONSOLE_DISP-3 -> /CONSOLE_DISP-1
- J5 pad 5: GND -> +3V3
- J6 pad 1: +3V3 -> GND
- J6 pad 2: /ADMIN_JOYSTICK-BUTTON -> /ADMIN_JOYSTICK-Y
- J6 pad 4: /ADMIN_JOYSTICK-Y -> /ADMIN_JOYSTICK-BUTTON
- J6 pad 5: GND -> +3V3
- J9 pad 1: /PUL+1 -> GND
- J9 pad 2: /DIR+1 -> /ENA+1
- J9 pad 3: /ENA+1 -> /DIR+1
- J9 pad 4: GND -> /PUL+1
- U1 pad 1: /IR_IN_2-dir -> /PA0
- U1 pad 3: /IR_IN_1-dir -> GND
- U1 pad 4: /IR_IN_1 -> /PA0
Routing:
- net /NRST: track 0.00 -> 73.5 mm, vias 0 -> 3
- net /IR_IN_2: track 0.00 -> 47.2 mm, vias 0 -> 2
- net /IR_IN_1: track 0.00 -> 40.9 mm, vias 0 -> 2
- net /PC13: track 0.00 -> 39.8 mm, vias 0 -> 1
- net /PA13: track 0.00 -> 36.1 mm, vias 0 -> 1
- net /PA14: track 0.00 -> 34.7 mm, vias 0 -> 1
- net /ADMIN_JOYSTICK-BUTTON: track 0.00 -> 34.2 mm, vias 0 -> 1
- net /PA9: track 0.00 -> 34.0 mm
- net /PC3: track 0.00 -> 33.5 mm, vias 0 -> 1
- net /PA8: track 0.00 -> 32.7 mm
- net /PB2: track 0.00 -> 31.8 mm, vias 0 -> 2
- net /G1: track 0.00 -> 30.9 mm
- net /ADMIN_JOYSTICK-X: track 0.00 -> 30.4 mm
- net /ADMIN_JOYSTICK-Y: track 0.00 -> 30.2 mm
- net /PC9: track 0.00 -> 30.2 mm
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- added copper zone on B.Cu, net GND
- removed copper zone on F.Cu, net /usbc-shield
Other:
- board size 64.8 x 61.5 mm -> 67.2 x 67.2 mm

Commit message: cleaned up
Parts:
- C20, C21: value 12.5pF -> 15pF
- FT1: value ~ -> FT232
- J1: footprint General Library:jtag_conn -> Sr_ Design:jtag_conn
- U1, U10, U4, U9: footprint General Library:KMR241G-RESET-BUTTON -> kicad_library:KMR241G-RESET-BUTTON
- U5: footprint kicad_library:TVS-DIODE-USBLC6-2SC6Y -> Sr_ Design:TVS-DIODE-USBLC6-2SC6Y
- XTAL2: value 8MHz(8PF) -> 8MHz(15pF)
- moved C23 28.7 mm to (79.1, 47.6)
- moved R9 28.6 mm to (81.3, 49.6)
- moved C13 28.6 mm to (59.6, 51.5)
- moved C21 28.6 mm to (67.7, 65.6)
- moved C3 28.6 mm to (39.5, 64.9)
- moved J11 28.6 mm to (77.9, 40.9)
- moved R20 28.6 mm to (55.1, 44.0)
- moved R8 28.6 mm to (48.4, 71.1)
- moved SW3 28.6 mm to (48.9, 82.3)
- moved U9 28.6 mm to (67.0, 51.6)
- moved XTAL1 28.6 mm to (61.9, 71.1)
- moved C1 28.6 mm to (29.5, 55.2)
- moved C12 28.6 mm to (59.8, 60.8)
- moved C16 28.6 mm to (51.5, 44.2)
- moved C17 28.6 mm to (46.7, 59.4)
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Routing:
- net GND: track 24.4 -> 49.0 mm, vias 27 -> 34
- net +5V: track 56.1 -> 68.2 mm
- net /V3.3_IN: track 0.00 -> 2.54 mm
- net /PA13: track 36.1 -> 33.9 mm
- net /PA14: track 34.7 -> 36.3 mm
- added copper zone on In1.Cu, net GND

Commit message: reorganized
updated + finished reorg
added footprints
added 2x8 jtag 3d file
Parts:
- J11: footprint Connector_PinSocket_2.54mm:PinSocket_2x08_P2.54mm_Vertical -> kicad_library:jst-02x08 conn
- moved R20 7.97 mm to (58.0, 36.6), turned to 180 degrees
- moved J11 5.58 mm to (80.2, 35.9), turned to 180 degrees
- moved R21 5.37 mm to (58.0, 32.4)
- moved LD4 3.43 mm to (53.7, 36.6), turned to 0 degrees
- moved LD5 1.52 mm to (53.6, 32.4), turned to 0 degrees
Routing:
- net /PB15: track 11.9 -> 22.0 mm
- net /A: track 19.6 -> 27.7 mm
- net /C: track 17.4 -> 25.1 mm
- net /PA4: track 28.9 -> 36.3 mm
- net /PA7: track 23.8 -> 31.2 mm
- net /B2: track 22.3 -> 29.4 mm
- net /B1: track 26.7 -> 33.8 mm
- net /CLK: track 17.5 -> 24.4 mm
- net /OE: track 17.5 -> 24.4 mm
- net /PC3: track 33.8 -> 37.8 mm
- net /B: track 21.4 -> 23.6 mm
- net /D: track 19.7 -> 21.2 mm
- net /G1: track 30.9 -> 31.8 mm
- net /G2: track 26.6 -> 27.6 mm
- net /LAT: track 20.6 -> 21.5 mm
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